Commit message: 20240412

File: my_niryo_robot_description/urdf/ned/niryo_ned_robot.urdf.xacro (robot description, xacro)
@@ -52,4 +52,9 @@
       <xacro:box_inertia m="10" x="1.1" y="0.7" z="0.03"/>
     </inertial>
+    <collision>
+      <geometry>
+        <box size="1.1 0.7 0.03" />
+      </geometry>
+    </collision>
   </link>
   <joint name="baseplate_joint" type="fixed">

File: my_niryo_robot_description/urdf/ned2/niryo_ned2_robot.urdf.xacro (robot description, xacro)
@@ -52,4 +52,9 @@
       <xacro:box_inertia m="10" x="1.1" y="0.7" z="0.03"/>
     </inertial>
+    <collision>
+      <geometry>
+        <box size="1.1 0.7 0.03" />
+      </geometry>
+    </collision>
   </link>
   <joint name="baseplate_joint" type="fixed">
